File: KiCad/First_PCb/Display.kicad_sch (KiCad schematic)
At the start: 7 parts, among them J1 Conn_01x04_Socket, J2 Conn_01x04_Socket, J3 Conn_01x04_Socket

Commit message: added all the kicad files & gerbers of the first pcb
Connections:
- net ESP_2ND_PCB_GPIO4 is gone; now on net GND: J2.1 (Pin_1)
- net +12V: now also J1.1 (Pin_1); no longer J3.3 (Pin_3)
- net +3.3V: now also J2.2 (Pin_2); no longer J1.3 (Pin_3)
- net ESP_LEDS_CLK: now also J1.3 (Pin_3); no longer J1.1 (Pin_1)
- net ESP_LEDS_SDI1: now also J3.1 (Pin_1); no longer J1.2 (Pin_2)
- net ESP_LEDS_SDI2: now also J3.2 (Pin_2); no longer J2.2 (Pin_2)
- net ESP_LEDS_SDI3: now also J3.3 (Pin_3); no longer J3.2 (Pin_2)
- net ESP_LEDS_SDI4: now also J1.2 (Pin_2); no longer J3.1 (Pin_1)
- net GND: no longer J2.4 (Pin_4)
- new net ESP_2ND_PCB_GPIO23: J2.4 (Pin_4)
Changed lines of the file:
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@@
-	(wire
-		(pts
-			(xy 87.63 81.28) (xy 124.46 81.28)
-		)
-		(stroke
-			(width 0)
-			(type default)
-		)
-	)
 	(wire
 		(pts
@@
 	(wire
 		(pts
-			(xy 118.11 102.87) (xy 124.46 102.87)
-		)
-		(stroke
-			(width 0)
-			(type default)
-		)
-	)
-	(wire
-		(pts
 			(xy 87.63 66.04) (xy 124.46 66.04)
 		)
@@
 	(wire
 		(pts
+			(xy 87.63 102.87) (xy 124.46 102.87)
+		)
+		(stroke
+			(width 0)
+			(type default)
+		)
+	)
+	(wire
+		(pts
+			(xy 104.14 81.28) (xy 124.46 81.28)
+		)
+		(stroke
+			(width 0)
+			(type default)
+		)
+	)
+	(wire
+		(pts
 			(xy 83.82 129.54) (xy 85.09 129.54)
 		)
@@
 		)
 	)
-	(hierarchical_label "ESP_LEDS_SDI1"
+	(hierarchical_label "ESP_LEDS_CLK"
 		(shape input)
-		(at 87.63 66.04 180)
+		(at 118.11 68.58 180)
 		(effects
 			(font
@@
 		)
 	)
-	(hierarchical_label "ESP_LEDS_CLK"
+	(hierarchical_label "ESP_LEDS_SDI1"
 		(shape input)
-		(at 87.63 63.5 180)
+		(at 87.63 97.79 180)
 		(effects
 			(font
@@
 		)
 	)
-	(hierarchical_label "ESP_LEDS_SDI3"
+	(hierarchical_label "ESP_LEDS_SDI2"
 		(shape input)
 		(at 87.63 100.33 180)
@@
 		)
 	)
-	(hierarchical_label "ESP_LEDS_SDI2"
+	(hierarchical_label "ESP_2ND_PCB_GPIO23"
 		(shape input)
-		(at 87.63 83.82 180)
+		(at 118.11 88.9 180)
 		(effects
 			(font
@@
 		)
 	)
-	(hierarchical_label "ESP_2ND_PCB_GPIO4"
+	(hierarchical_label "ESP_LEDS_SDI4"
 		(shape input)
-		(at 87.63 81.28 180)
+		(at 87.63 66.04 180)
 		(effects
 			(font
@@
 		)
 	)
-	(hierarchical_label "ESP_LEDS_SDI4"
+	(hierarchical_label "ESP_LEDS_SDI3"
 		(shape input)
-		(at 87.63 97.79 180)
+		(at 87.63 102.87 180)
 		(effects
 			(font
@@
 	(symbol
 		(lib_id "power:+5V")
-		(at 118.11 102.87 0)
+		(at 87.63 63.5 0)
 		(unit 1)
 		(exclude_from_sim no)
@@
 		(dnp no)
 		(property "Reference" "#PWR022"
-			(at 118.11 106.68 0)
+			(at 87.63 67.31 0)
 			(effects
 				(font
@@
 		)
 		(property "Value" "+12V"
-			(at 114.808 102.616 0)
+			(at 84.328 63.246 0)
 			(effects
 				(font
@@
 		)
 		(property "Footprint" ""
-			(at 118.11 102.87 0)
+			(at 87.63 63.5 0)
 			(effects
 				(font
@@
 		)
 		(property "Datasheet" ""
-			(at 118.11 102.87 0)
+			(at 87.63 63.5 0)
 			(effects
 				(font
@@
 		)
 		(property "Description" "Power symbol creates a global label with name \"+5V\""
-			(at 118.11 102.87 0)
+			(at 87.63 63.5 0)
 			(effects
 				(font
@@
 	(symbol
 		(lib_id "power:+5V")
-		(at 118.11 68.58 0)
+		(at 87.63 83.82 0)
 		(unit 1)
 		(exclude_from_sim no)
@@
 		(dnp no)
 		(property "Reference" "#PWR026"
-			(at 118.11 72.39 0)
+			(at 87.63 87.63 0)
 			(effects
 				(font
@@
 		)
 		(property "Value" "+3.3V"
-			(at 114.808 67.818 0)
+			(at 84.328 83.058 0)
 			(effects
 				(font
@@
 		)
 		(property "Footprint" ""
-			(at 118.11 68.58 0)
+			(at 87.63 83.82 0)
 			(effects
 				(font
@@
 		)
 		(property "Datasheet" ""
-			(at 118.11 68.58 0)
+			(at 87.63 83.82 0)
 			(effects
 				(font
@@
 		)
 		(property "Description" "Power symbol creates a global label with name \"+5V\""
-			(at 118.11 68.58 0)
+			(at 87.63 83.82 0)
 			(effects
 				(font
@@
 	(symbol
 		(lib_id "power:GND")
-		(at 118.11 88.9 0)
+		(at 104.14 81.28 0)
 		(unit 1)
 		(exclude_from_sim no)
@@
 		(dnp no)
 		(property "Reference" "#PWR023"
-			(at 118.11 95.25 0)
+			(at 104.14 87.63 0)
 			(effects
 				(font
@@
 		)
 		(property "Value" "GND"
-			(at 114.808 91.44 0)
+			(at 100.838 83.82 0)
 			(effects
 				(font
@@
 		)
 		(property "Footprint" ""
-			(at 118.11 88.9 0)
+			(at 104.14 81.28 0)
 			(effects
 				(font
@@
 		)
 		(property "Datasheet" ""
-			(at 118.11 88.9 0)
+			(at 104.14 81.28 0)
 			(effects
 				(font
@@
 		)
 		(property "Description" "Power symbol creates a global label with name \"GND\" , ground"
-			(at 118.11 88.9 0)
-			(effects
-				(font
+			(at 104.14 81.28 0)
+			(effects
+				(font
