File: KiCad/Second_PCB/2ND_PCB.kicad_sch (KiCad schematic)
At the start: 8 parts

Commit message: added all the kicad files and gerbers of the second pcb
after sending to manufacture.
Parts:
- removed R1, R2, R3: 10, Resistor_SMD:R_0603_1608Metric_Pad0.98x0.95mm_HandSolder, symbol Device:R
Connections:
- net ESP_2ND_PCB_GPIO4 renamed ESP_2ND_PCB_GPIO23
- no-connect marks 4 -> 0
Other:
- sheet 10_LED_ARM1 ports: added none; removed SDO1
- sheet 10_LED_ARM2 ports: added none; removed SDO2
- sheet 10_LED_ARM3 ports: added none; removed SDO3
- sheet 10_LED_ARM4 ports: added none; removed SDO4
