File: KiCad/Second_PCB/LOWER_PCB_CONNECTORS.kicad_sch (KiCad schematic)
At the start: 3 parts, among them J1 Conn_01x04_Pin, J2 Conn_01x04_Pin, J3 Conn_01x04_Pin

Commit message: added all the kicad files and gerbers of the second pcb
after sending to manufacture.
Parts:
- J1, J2, J3: footprint Connector_PinHeader_2.54mm:PinHeader_1x04_P2.54mm_Vertical -> Connector_PinSocket_2.54mm:PinSocket_1x04_P2.54mm_Vertical
Connections:
- net +12V: now also J1.1 (Pin_1); no longer J3.3 (Pin_3)
- net +3.3V: now also J2.2 (Pin_2); no longer J1.3 (Pin_3)
- net ESP_2ND_PCB_GPIO4: now also J2.4 (Pin_4); no longer J2.1 (Pin_1)
- net ESP_LEDS_CLK: now also J1.3 (Pin_3); no longer J1.1 (Pin_1)
- net ESP_LEDS_SDI1: now also J3.1 (Pin_1); no longer J1.2 (Pin_2)
- net ESP_LEDS_SDI2: now also J3.2 (Pin_2); no longer J2.2 (Pin_2)
- net ESP_LEDS_SDI3: now also J3.3 (Pin_3); no longer J3.2 (Pin_2)
- net ESP_LEDS_SDI4: now also J1.2 (Pin_2); no longer J3.1 (Pin_1)
- net GND: now also J2.1 (Pin_1); no longer J2.4 (Pin_4)
Changed lines of the file:
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@@
-	(wire
-		(pts
-			(xy 114.3 71.12) (xy 148.59 71.12)
-		)
-		(stroke
-			(width 0)
-			(type default)
-		)
-	)
 	(wire
 		(pts
@@
 	(wire
 		(pts
-			(xy 114.3 78.74) (xy 121.92 78.74)
-		)
-		(stroke
-			(width 0)
-			(type default)
-		)
-	)
-	(wire
-		(pts
-			(xy 114.3 73.66) (xy 148.59 73.66)
-		)
-		(stroke
-			(width 0)
-			(type default)
-		)
-	)
-	(wire
-		(pts
-			(xy 114.3 96.52) (xy 121.92 96.52)
+			(xy 114.3 78.74) (xy 139.7 78.74)
+		)
+		(stroke
+			(width 0)
+			(type default)
+		)
+	)
+	(wire
+		(pts
+			(xy 114.3 73.66) (xy 139.7 73.66)
+		)
+		(stroke
+			(width 0)
+			(type default)
+		)
+	)
+	(wire
+		(pts
+			(xy 114.3 96.52) (xy 148.59 96.52)
 		)
 		(stroke
@@
 	(wire
 		(pts
-			(xy 114.3 53.34) (xy 148.59 53.34)
-		)
-		(stroke
-			(width 0)
-			(type default)
-		)
-	)
-	(wire
-		(pts
-			(xy 114.3 50.8) (xy 148.59 50.8)
+			(xy 114.3 53.34) (xy 147.32 53.34)
+		)
+		(stroke
+			(width 0)
+			(type default)
+		)
+	)
+	(wire
+		(pts
+			(xy 114.3 50.8) (xy 147.32 50.8)
 		)
 		(stroke
@@
 	(wire
 		(pts
-			(xy 114.3 55.88) (xy 121.92 55.88)
-		)
-		(stroke
-			(width 0)
-			(type default)
-		)
-	)
-	(hierarchical_label "ESP_LEDS_SDI3"
+			(xy 114.3 55.88) (xy 147.32 55.88)
+		)
+		(stroke
+			(width 0)
+			(type default)
+		)
+	)
+	(wire
+		(pts
+			(xy 114.3 71.12) (xy 133.35 71.12)
+		)
+		(stroke
+			(width 0)
+			(type default)
+		)
+	)
+	(hierarchical_label "ESP_LEDS_SDI4"
+		(shape output)
+		(at 147.32 53.34 0)
+		(effects
+			(font
+				(size 1.27 1.27)
+			)
+			(justify left)
+		)
+	)
+	(hierarchical_label "ESP_LEDS_CLK"
+		(shape output)
+		(at 147.32 55.88 0)
+		(effects
+			(font
+				(size 1.27 1.27)
+			)
+			(justify left)
+		)
+	)
+	(hierarchical_label "ESP_LEDS_SDI2"
 		(shape output)
 		(at 148.59 93.98 0)
@@
 		)
 	)
-	(hierarchical_label "ESP_LEDS_SDI2"
-		(shape output)
-		(at 148.59 73.66 0)
-		(effects
-			(font
-				(size 1.27 1.27)
-			)
-			(justify left)
-		)
-	)
 	(hierarchical_label "ESP_LEDS_SDI1"
-		(shape output)
-		(at 148.59 53.34 0)
-		(effects
-			(font
-				(size 1.27 1.27)
-			)
-			(justify left)
-		)
-	)
-	(hierarchical_label "ESP_LEDS_CLK"
-		(shape output)
-		(at 148.59 50.8 0)
-		(effects
-			(font
-				(size 1.27 1.27)
-			)
-			(justify left)
-		)
-	)
-	(hierarchical_label "ESP_2ND_PCB_GPIO4"
-		(shape output)
-		(at 148.59 71.12 0)
-		(effects
-			(font
-				(size 1.27 1.27)
-			)
-			(justify left)
-		)
-	)
-	(hierarchical_label "ESP_LEDS_SDI4"
 		(shape output)
 		(at 148.59 91.44 0)
@@
 		)
 	)
+	(hierarchical_label "ESP_2ND_PCB_GPIO4"
+		(shape output)
+		(at 139.7 78.74 0)
+		(effects
+			(font
+				(size 1.27 1.27)
+			)
+			(justify left)
+		)
+	)
+	(hierarchical_label "ESP_LEDS_SDI3"
+		(shape output)
+		(at 148.59 96.52 0)
+		(effects
+			(font
+				(size 1.27 1.27)
+			)
+			(justify left)
+		)
+	)
 	(symbol
 		(lib_id "Connector:Conn_01x04_Pin")
@@
 			)
 		)
-		(property "Footprint" "Connector_PinHeader_2.54mm:PinHeader_1x04_P2.54mm_Vertical"
+		(property "Footprint" "Connector_PinSocket_2.54mm:PinSocket_1x04_P2.54mm_Vertical"
 			(at 109.22 73.66 0)
 			(effects
@@
 			)
 		)
-		(property "Footprint" "Connector_PinHeader_2.54mm:PinHeader_1x04_P2.54mm_Vertical"
+		(property "Footprint" "Connector_PinSocket_2.54mm:PinSocket_1x04_P2.54mm_Vertical"
 			(at 109.22 93.98 0)
 			(effects
@@
 			)
 		)
-		(property "Footprint" "Connector_PinHeader_2.54mm:PinHeader_1x04_P2.54mm_Vertical"
+		(property "Footprint" "Connector_PinSocket_2.54mm:PinSocket_1x04_P2.54mm_Vertical"
 			(at 109.22 53.34 0)
 			(effects
@@
 	(symbol
 		(lib_id "power:+3.3V")
-		(at 121.92 55.88 0)
+		(at 139.7 73.66 0)
 		(unit 1)
 		(exclude_from_sim no)
@@
 		(dnp no)
 		(property "Reference" "#PWR085"
-			(at 121.92 59.69 0)
+			(at 139.7 77.47 0)
 			(effects
 				(font
@@
 		)
 		(property "Value" "+3.3V"
-			(at 125.222 55.372 0)
+			(at 143.002 73.152 0)
 			(effects
 				(font
@@
 		)
 		(property "Footprint" ""
-			(at 121.92 55.88 0)
+			(at 139.7 73.66 0)
 			(effects
 				(font
@@
 		)
 		(property "Datasheet" ""
-			(at 121.92 55.88 0)
+			(at 139.7 73.66 0)
 			(effects
 				(font
@@
 		)
 		(property "Description" "Power symbol creates a global label with name \"+3.3V\""
-			(at 121.92 55.88 0)
-			(effects
-				(font
-					(size 1.27 1.27)
-				)
-				(hide yes)
-			)
-		)
-		(pin "1"
-		)
-		(instances
-			(project ""
+			(at 139.7 73.66 0)
+			(effects
+				(font
+					(size 1.27 1.27)
+				)
+				(hide yes)
+			)
+		)
+		(pin "1"
+		)
+		(instances
+			(project "2ND_PCB"
 				(path "/500a9f84-d59e-418d-bc4b-2142a90d742d/cfbbf487-0da7-4357-bd55-3c8e5524ea6e"
 					(reference "#PWR085")
@@
 	(symbol
 		(lib_id "power:GND")
-		(at 121.92 78.74 0)
+		(at 133.35 71.12 0)
 		(unit 1)
 		(exclude_from_sim no)
@@
 		(fields_autoplaced yes)
 		(property "Reference" "#PWR012"
-			(at 121.92 85.09 0)
+			(at 133.35 77.47 0)
 			(effects
 				(font
@@
 		)
 		(property "Value" "GND"
-			(at 121.92 83.82 0)
+			(at 133.35 76.2 0)
 			(effects
 				(font
@@
 		)
 		(property "Footprint" ""
-			(at 121.92 78.74 0)
+			(at 133.35 71.12 0)
 			(effects
 				(font
@@
 		)
 		(property "Datasheet" ""
-			(at 121.92 78.74 0)
+			(at 133.35 71.12 0)
 			(effects
 				(font
@@
 		)
 		(property "Description" "Power symbol creates a global label with name \"GND\" , ground"
-			(at 121.92 78.74 0)
+			(at 133.35 71.12 0)
 			(effects
 				(font
@@
 	(symbol
 		(lib_id "power:+12V")
-		(at 121.92 96.52 0)
+		(at 147.32 50.8 0)
 		(unit 1)
 		(exclude_from_sim no)
@@
 		(dnp no)
 		(property "Reference" "#PWR084"
-			(at 121.92 100.33 0)
+			(at 147.32 54.61 0)
 			(effects
 				(font
@@
 		)
 		(property "Value" "+12V"
-			(at 125.222 96.012 0)
+			(at 150.622 50.292 0)
 			(effects
 				(font
@@
 		)
 		(property "Footprint" ""
-			(at 121.92 96.52 0)
+			(at 147.32 50.8 0)
 			(effects
 				(font
@@
 		)
 		(property "Datasheet" ""
-			(at 121.92 96.52 0)
+			(at 147.32 50.8 0)
 			(effects
 				(font
@@
 		)
 		(property "Description" "Power symbol creates a global label with name \"+12V\""
-			(at 121.92 96.52 0)
-			(effects
-				(font
-					(size 1.27 1.27)
-				)
-				(hide yes)
-			)
-		)
-		(pin "1"
-		)
-		(instances
-			(project ""
+			(at 147.32 50.8 0)
+			(effects
+				(font
+					(size 1.27 1.27)
+				)
+				(hide yes)
+			)
+		)
+		(pin "1"
+		)
+		(instances
+			(project "2ND_PCB"
 				(path "/500a9f84-d59e-418d-bc4b-2142a90d742d/cfbbf487-0da7-4357-bd55-3c8e5524ea6e"
 					(reference "#PWR084")
